File: circuitry/auxiliary.kicad_sch (KiCad schematic)
At the start: 17 parts, among them P31 JST XH 3pin, P32 JST XH 3pin, P33 JST XH 3pin, P34 JST XH 3pin

Commit message: feat: Add sensors & structure main program
Parts:
- S1: value DS1307 + AT24C32 -> DS3231 + AT24C32
Changed lines of the file:
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@@
 			)
 		)
-		(property "Value" "DS1307 + AT24C32"
+		(property "Value" "DS3231 + AT24C32"
 			(at 203.2 19.812 0)
 			(show_name no)
