File: circuitry/circuit.kicad_sch (KiCad schematic)
At the start: 43 parts, among them P1 45A Anderson PowerPole, P10 JST XH 2pin, P11 JST XH 2pin, P12 JST XH 2pin, P13 JST XH 2pin, P14 JST XH 2pin, P15 JST XH 2pin, P16 JST XH 2pin, P17 JST XH 2pin, P18 JST XH 2pin, P19 JST XH 2pin, P2 45A Anderson PowerPole, P20 JST XH 2pin, P21 JST XH 2pin, P22 JST XH 2pin, P23 JST XH 2pin, P24 JST XH 2pin, P25 JST XH 2pin, P26 JST XH 2pin, P27 JST XH 3pin, P28 JST XH 3pin, P29 JST XH 3pin, P3 45A Anderson PowerPole, P30 JST XH 3pin, P4 45A Anderson PowerPole, P5 45A Anderson PowerPole, P6 45A Anderson PowerPole, P9 JST XH 2pin, SW1 6A Momentary, SW2 6A SPDT, SW3 6A SPDT, SW4 6A Momentary SPDT, SW5 SPDT

Commit message: fix: Resolve circuit signal issues
Parts:
- F1: value 2A -> 4A
Changed lines of the file:
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@@
 		(title "Main Circuit Diagram")
 		(date "2026-06-28")
-		(rev "3")
+		(rev "4")
 		(company "Wackadoos F24+")
 		(comment 1 "Connector Convention: Pin 1 = GND. Pin 2 = VCC. Further pins are signal")
@@
 			)
 		)
-		(property "Value" "2A"
+		(property "Value" "4A"
 			(at 35.306 177.546 90)
 			(show_name no)

Commit message: fix: Revise circuit plugs & resistors
Parts:
- removed P25: JST XH 2pin, symbol Connector:Conn_01x02_Socket
- removed P26: JST XH 2pin, symbol Connector:Conn_01x02_Pin
- removed P27, P30: JST XH 3pin, symbol Connector:Conn_01x03_Pin
- removed P28, P29: JST XH 3pin, symbol Connector:Conn_01x03_Socket
- removed P5: 45A Anderson PowerPole, symbol Connector:Conn_01x02_Socket
- removed P6: 45A Anderson PowerPole, symbol Connector:Conn_01x02_Pin
- P21: Friendly Name (Dashboard) -> (Power Panel)
- P22: Friendly Name (Instruments Box) -> (Instruments Loom)
Connections:
- net Motor Housing/FAN: now also P24.2 (Pin_2)
- net Motor Housing/KILL: now also P24.1 (Pin_1)
Other:
- note removed: "BRAKE LIGHT"
- note removed: "BRAKE SWITCH"
- note removed: "ESC LOOM A"
- note removed: "ESC LOOM B"
- note removed: "ESC POWER"
- note removed: "HORN"
- note removed: "INSTRUMENTS POWER"
- note removed: "MAIN BATTERY"
- moved on the sheet: P23, P24
