File: circuitry/drive.kicad_sch (KiCad schematic)
At the start: 16 parts, among them M1 105ZDY08, M2 12025, M3 9733, P35 JST XH 4pin, P36 JST XH 4pin, P37 JST XH 4pin, P38 JST XH 4pin, P7 45A Anderson PowerPole, P8 45A Anderson PowerPole

Commit message: fix: Revise circuit plugs & resistors
Parts:
- added P25, P43, P45: JST XH 2pin, symbol Connector:Conn_01x02_Socket
- added P26, P44, P46: JST XH 2pin, symbol Connector:Conn_01x02_Pin
- added P29, P40, P42: JST XH 3pin, symbol Connector:Conn_01x03_Socket
- added P30, P39, P41: JST XH 3pin, symbol Connector:Conn_01x03_Pin
- added P5: 45A Anderson PowerPole, symbol Connector:Conn_01x02_Socket
- added P6: 45A Anderson PowerPole, symbol Connector:Conn_01x02_Pin
Connections:
- net FAN: now also P25.2 (Pin_2); no longer M2.1 (+), M3.1 (+)
- net KILL: now also P25.1 (Pin_1); no longer ESC1.6 (SERVO), R3.2
- net RX: now also P29.2 (Pin_2); no longer ESC1.22 (RX/SDA)
- net TEMP: now also P29.3 (Pin_3); no longer S6.2 (DQ), S7.2 (DQ)
- net TX: now also P29.1 (Pin_1); no longer ESC1.21 (TX/SCL)
- net VBAT+: now also P5.2 (Pin_2); no longer ESC1.1 (VBAT+)
- net VBAT-: now also P5.1 (Pin_1); no longer ESC1.2 (VBAT-), M2.2 (-), M3.2 (-)
- net at R3.1: now also ESC1.6 (SERVO), P26.1 (Pin_1); no longer ESC1.16 (3.3v)
- new net: ESC1.21 (TX/SCL), P30.1 (Pin_1)
- new net: ESC1.22 (RX/SDA), P30.2 (Pin_2)
- new net: P30.3 (Pin_3), P39.3 (Pin_3), P41.3 (Pin_3)
- new net: ESC1.8 (GND), P39.1 (Pin_1), P41.1 (Pin_1)
- new net: ESC1.7 (5v), P39.2 (Pin_2), P41.2 (Pin_2)
- new net: M2.2 (-), P44.1 (Pin_1)
- new net: M2.1 (+), P44.2 (Pin_2)
- new net: P40.1 (Pin_1), S6.1 (GND)
- new net: P40.2 (Pin_2), S6.3 (VDD)
- new net: P40.3 (Pin_3), S6.2 (DQ)
- new net: P45.1 (Pin_1), P6.1 (Pin_1)
- new net: P26.2 (Pin_2), P43.2 (Pin_2), P45.2 (Pin_2)
- new net: P42.1 (Pin_1), S7.1 (GND)
- new net: P42.2 (Pin_2), S7.3 (VDD)
- new net: P42.3 (Pin_3), S7.2 (DQ)
- new net: M3.1 (+), P46.2 (Pin_2)
- new net: M3.2 (-), P46.1 (Pin_1)
- new net: ESC1.1 (VBAT+), P6.2 (Pin_2)
- new net: ESC1.16 (3.3v), R3.2
- new net: ESC1.2 (VBAT-), P43.1 (Pin_1)
Other:
- note removed: "CONTROLS LOOM"
- note removed: "MAIN MOTOR"
- moved on the sheet: M1, P7, P8, S6, S7
